Commit message: add door room, add collisions of jaco arm, add gazebo grasp_fix plugin

File: qm_description/urdf/manipulator/common/kinova_common.xacro (robot description, xacro)
@@ -15,5 +15,5 @@
 <xacro:include filename="$(find qm_description)/urdf/manipulator/common/kinova_inertial.xacro" />
     <xacro:property name="J_PI" value="3.1415926535897931" />
-    <xacro:macro name="kinova_armlink" params="link_name link_mesh ring_mesh:=ring_big use_ring_mesh:=false mesh_no col:=false">
+    <xacro:macro name="kinova_armlink" params="link_name link_mesh ring_mesh:=ring_big use_ring_mesh:=false mesh_no col:=true">
       <link name="${link_name}">
           <visual>

File: qm_description/urdf/manipulator/j2n6s300.xacro (robot description, xacro)
@@ -120,5 +120,5 @@
         <xacro:kinova_virtual_link link_name="${prefix}_end_effector"/>
         <xacro:kinova_virtual_joint joint_name="${prefix}_joint_end_effector" type="${joint_end_effector_type}" parent="${prefix}_link_6" child="${prefix}_end_effector" joint_axis_xyz="${joint_end_effector_axis_xyz}" joint_origin_xyz="${joint_end_effector_origin_xyz}" joint_origin_rpy="${joint_end_effector_origin_rpy}" joint_lower_limit="0" joint_upper_limit="0"/>
-    <xacro:kinova_3fingers link_hand="${prefix}_link_6" prefix="${prefix}_"/>
+        <xacro:kinova_3fingers link_hand="${prefix}_link_6" prefix="${prefix}_"/>
     </xacro:macro>
 </root>

File: qm_description/urdf/manipulator/j2n6s300fix.xacro (robot description, xacro)
@@ -120,5 +120,5 @@
         <xacro:kinova_virtual_link link_name="${prefix}_end_effector"/>
         <xacro:kinova_virtual_joint joint_name="${prefix}_joint_end_effector" type="${joint_end_effector_type}" parent="${prefix}_link_6" child="${prefix}_end_effector" joint_axis_xyz="${joint_end_effector_axis_xyz}" joint_origin_xyz="${joint_end_effector_origin_xyz}" joint_origin_rpy="${joint_end_effector_origin_rpy}" joint_lower_limit="0" joint_upper_limit="0"/>
-<!--     <xacro:kinova_3fingers link_hand="${prefix}_link_6" prefix="${prefix}_"/> -->
+        <xacro:kinova_3fingers link_hand="${prefix}_link_6" prefix="${prefix}_"/>
     </xacro:macro>
 </root>

File: qm_description/urdf/quadruped_manipulator/robot.xacro (robot description, xacro)
@@ -5,4 +5,5 @@
     <xacro:include filename="$(find qm_description)/urdf/quadruped/robot.xacro" />
     <!-- manipulatior -->
+    <!--xacro:include filename="$(find qm_description)/urdf/manipulator/j2n6s300fix.xacro"/-->
     <xacro:include filename="$(find qm_description)/urdf/manipulator/j2n6s300fix.xacro"/>
     <link name="arm_base_link" />

Commit message: add door_world without wall

File: qm_description/urdf/manipulator/common/kinova_common.xacro (robot description, xacro)
@@ -15,5 +15,5 @@
 <xacro:include filename="$(find qm_description)/urdf/manipulator/common/kinova_inertial.xacro" />
     <xacro:property name="J_PI" value="3.1415926535897931" />
-    <xacro:macro name="kinova_armlink" params="link_name link_mesh ring_mesh:=ring_big use_ring_mesh:=false mesh_no col:=true">
+    <xacro:macro name="kinova_armlink" params="link_name link_mesh ring_mesh:=ring_big use_ring_mesh:=false mesh_no col:=false">
       <link name="${link_name}">
           <visual>

File: qm_description/urdf/manipulator/j2n6s300fix.xacro (robot description, xacro)
@@ -120,5 +120,5 @@
         <xacro:kinova_virtual_link link_name="${prefix}_end_effector"/>
         <xacro:kinova_virtual_joint joint_name="${prefix}_joint_end_effector" type="${joint_end_effector_type}" parent="${prefix}_link_6" child="${prefix}_end_effector" joint_axis_xyz="${joint_end_effector_axis_xyz}" joint_origin_xyz="${joint_end_effector_origin_xyz}" joint_origin_rpy="${joint_end_effector_origin_rpy}" joint_lower_limit="0" joint_upper_limit="0"/>
-        <xacro:kinova_3fingers link_hand="${prefix}_link_6" prefix="${prefix}_"/>
+        <!-- <xacro:kinova_3fingers link_hand="${prefix}_link_6" prefix="${prefix}_"/> -->
     </xacro:macro>
 </root>

Commit message: add gripper & whole body collision

File: qm_description/urdf/manipulator/common/kinova_common.xacro (robot description, xacro)
@@ -15,5 +15,6 @@
 <xacro:include filename="$(find qm_description)/urdf/manipulator/common/kinova_inertial.xacro" />
     <xacro:property name="J_PI" value="3.1415926535897931" />
-    <xacro:macro name="kinova_armlink" params="link_name link_mesh ring_mesh:=ring_big use_ring_mesh:=false mesh_no col:=false">
+    <!-- Modify collision value here: col:=true/false -->
+    <xacro:macro name="kinova_armlink" params="link_name link_mesh ring_mesh:=ring_big use_ring_mesh:=false mesh_no col:=true">
       <link name="${link_name}">
           <visual>

File: qm_description/urdf/manipulator/j2n6s300fix.xacro (robot description, xacro)
@@ -120,5 +120,5 @@
         <xacro:kinova_virtual_link link_name="${prefix}_end_effector"/>
         <xacro:kinova_virtual_joint joint_name="${prefix}_joint_end_effector" type="${joint_end_effector_type}" parent="${prefix}_link_6" child="${prefix}_end_effector" joint_axis_xyz="${joint_end_effector_axis_xyz}" joint_origin_xyz="${joint_end_effector_origin_xyz}" joint_origin_rpy="${joint_end_effector_origin_rpy}" joint_lower_limit="0" joint_upper_limit="0"/>
-        <!-- <xacro:kinova_3fingers link_hand="${prefix}_link_6" prefix="${prefix}_"/> -->
+        <xacro:kinova_3fingers link_hand="${prefix}_link_6" prefix="${prefix}_"/>
     </xacro:macro>
 </root>

File: qm_description/urdf/quadruped_manipulator/robot.xacro (robot description, xacro)
@@ -5,5 +5,4 @@
     <xacro:include filename="$(find qm_description)/urdf/quadruped/robot.xacro" />
     <!-- manipulatior -->
-    <!--xacro:include filename="$(find qm_description)/urdf/manipulator/j2n6s300fix.xacro"/-->
     <xacro:include filename="$(find qm_description)/urdf/manipulator/j2n6s300fix.xacro"/>
     <link name="arm_base_link" />

File: qm_description/urdf/quadruped_manipulator/robot_mpc.xacro (robot description, xacro)
@@ -4,5 +4,5 @@
     <xacro:arg name="robot_type" default="aliengo"/>
     <xacro:include filename="$(find qm_description)/urdf/quadruped/robot.xacro" />
-    <!-- manipulatior -->
+    <!-- manipulator -->
     <xacro:include filename="$(find qm_description)/urdf/manipulator/j2n6s300fix.xacro"/>
     <link name="arm_base_link" />

Commit message: add stage1~3; change opening strategy: rotate handle and then ungrasp

File: qm_description/urdf/manipulator/common/kinova_common.xacro (robot description, xacro)
@@ -135,5 +135,6 @@
             <axis xyz="0 0 1"/>
             <origin xyz="${finger_origin_xyz}" rpy="${finger_origin_rpy}"/>
-            <limit lower="0" upper="1.51" effort="2" velocity="1"/>
+            <!-- <limit lower="0" upper="1.51" effort="2" velocity="1"/> -->
+            <limit lower="0" upper="1.51" effort="20" velocity="0.2"/>
         </joint>
 		    <transmission name="${prefix}joint_finger_${finger_number}_trans">
@@ -147,5 +148,6 @@
 					</actuator>
 		    </transmission>
-        <xacro:kinova_armlink link_name="${prefix}link_finger_tip_${finger_number}" link_mesh="finger_distal" mesh_no="58"/>
+        <!-- try grasping without finger_tip -->
+        <!-- <xacro:kinova_armlink link_name="${prefix}link_finger_tip_${finger_number}" link_mesh="finger_distal" mesh_no="58"/>
         <joint name="${prefix}joint_finger_tip_${finger_number}" type="revolute">
             <parent link="${prefix}link_finger_${finger_number}"/>
@@ -153,5 +155,5 @@
             <axis xyz="0 0 1"/>
             <origin xyz="0.044 -0.003 0" rpy="0 0 0"/>
-            <limit lower="0" upper="2" effort="2" velocity="1"/>
+            <limit lower="0" upper="2" effort="2" velocity="0.2"/>
         </joint>
         <transmission name="${prefix}joint_finger_tip_${finger_number}_trans">
@@ -164,5 +166,5 @@
 					<mechanicalReduction>1</mechanicalReduction>
 					</actuator>
-        </transmission>
+        </transmission> -->
     </xacro:macro>
 </root>

File: qm_description/urdf/manipulator/j2n6s300fix.xacro (robot description, xacro)
@@ -131,7 +131,7 @@
                 <gripper_link> j2n6s300_link_finger_2 </gripper_link>
                 <gripper_link> j2n6s300_link_finger_3 </gripper_link>
-                <gripper_link> j2n6s300_link_finger_tip_1 </gripper_link>
+                <!-- <gripper_link> j2n6s300_link_finger_tip_1 </gripper_link>
                 <gripper_link> j2n6s300_link_finger_tip_2 </gripper_link>
-                <gripper_link> j2n6s300_link_finger_tip_3 </gripper_link>
+                <gripper_link> j2n6s300_link_finger_tip_3 </gripper_link> -->
             </arm>
             <forces_angle_tolerance>100</forces_angle_tolerance>
@@ -140,5 +140,5 @@
             <max_grip_count>8</max_grip_count>
             <release_tolerance>0.01</release_tolerance>
-            <disable_collisions_on_attach>false</disable_collisions_on_attach>
+            <disable_collisions_on_attach>true</disable_collisions_on_attach>
             <contact_topic>__default_topic__</contact_topic>
         </plugin>

Commit message: push door but straight; problem on releasing handle

File: qm_description/urdf/manipulator/common/kinova_common.xacro (robot description, xacro)
@@ -136,5 +136,5 @@
             <origin xyz="${finger_origin_xyz}" rpy="${finger_origin_rpy}"/>
             <!-- <limit lower="0" upper="1.51" effort="2" velocity="1"/> -->
-            <limit lower="0" upper="1.51" effort="20" velocity="0.2"/>
+            <limit lower="0" upper="1.51" effort="200" velocity="0.2"/>
         </joint>
 		    <transmission name="${prefix}joint_finger_${finger_number}_trans">

File: qm_description/urdf/manipulator/j2n6s300fix.xacro (robot description, xacro)
@@ -131,7 +131,4 @@
                 <gripper_link> j2n6s300_link_finger_2 </gripper_link>
                 <gripper_link> j2n6s300_link_finger_3 </gripper_link>
-                <!-- <gripper_link> j2n6s300_link_finger_tip_1 </gripper_link>
-                <gripper_link> j2n6s300_link_finger_tip_2 </gripper_link>
-                <gripper_link> j2n6s300_link_finger_tip_3 </gripper_link> -->
             </arm>
             <forces_angle_tolerance>100</forces_angle_tolerance>
